Commit message: 让仿真机器人移动起来

File: src/zznbot_description/urdf/fishbot/actuator/caster.urdf.xacro (robot description, xacro)
@@ -36,4 +36,10 @@
             <origin xyz="${xyz}" rpy="0.0 0.0 0.0"/>
         </joint>
+        <gazebo reference="${caster_name}_link">
+            <mu1 value="0.0"/>
+            <mu1 value="0.0"/>
+            <kp value="1000000000.0"/>
+            <kd value="1.0"/>
+        </gazebo>
     </xacro:macro>
 </robot>

File: src/zznbot_description/urdf/fishbot/actuator/wheel.urdf.xacro (robot description, xacro)
@@ -37,4 +37,10 @@
             <axis xyz="0.0 1.0 0.0"/>
         </joint>
+        <gazebo reference="${wheel_name}_link">
+            <mu1 value="20.0"/>
+            <mu1 value="20.0"/>
+            <kp value="1000000000.0"/>
+            <kd value="1.0"/>
+        </gazebo>
     </xacro:macro>
 </robot>

File: src/zznbot_description/urdf/fishbot/fishbot.urdf.xacro (robot description, xacro)
@@ -10,4 +10,6 @@
 <xacro:include filename="$(find zznbot_description)/urdf/fishbot/actuator/wheel.urdf.xacro"/>
 <xacro:include filename="$(find zznbot_description)/urdf/fishbot/actuator/caster.urdf.xacro"/>
+<!-- 插件 -->
+<xacro:include filename="$(find zznbot_description)/urdf/fishbot/plugins/gazebo_control_plugin.xacro"/>
 <xacro:base_xacro length="0.12" radius="0.10"/>
 <xacro:imu_xacro xyz="0.0 0.0 0.02"/>
@@ -18,3 +20,4 @@
 <xacro:caster_xacro caster_name="front_caster" xyz="0.08 0.0 -0.076"/>
 <xacro:caster_xacro caster_name="back_caster" xyz="-0.08 0.0 -0.076"/>
+<xacro:gazebo_control_plugin/>
 </robot>

File: src/zznbot_description/urdf/fishbot/sensor/laser.urdf.xacro (robot description, xacro)
@@ -75,4 +75,10 @@
             <origin xyz="${xyz}" rpy="0.0 0.0 0.0"/>
         </joint>
+        <gazebo reference="laser_cylinder_link">
+            <material>Gazebo/Black</material>
+        </gazebo>
+        <gazebo reference="laser_link">
+            <material>Gazebo/Black</material>
+        </gazebo>
     </xacro:macro>
 </robot>
