Commit message: 20260317

File: src/zznbot_description/urdf/fishbot/fishbot.urdf.xacro (robot description, xacro)
@@ -12,4 +12,5 @@
 <!-- 插件 -->
 <xacro:include filename="$(find zznbot_description)/urdf/fishbot/plugins/gazebo_control_plugin.xacro"/>
+<xacro:include filename="$(find zznbot_description)/urdf/fishbot/plugins/gazebo_sensor_plugin.xacro"/>
 <xacro:base_xacro length="0.12" radius="0.10"/>
 <xacro:imu_xacro xyz="0.0 0.0 0.02"/>
@@ -21,3 +22,4 @@
 <xacro:caster_xacro caster_name="back_caster" xyz="-0.08 0.0 -0.076"/>
 <xacro:gazebo_control_plugin/>
+<xacro:gazebo_sensor_plugin/>
 </robot>

File: src/zznbot_description/urdf/fishbot/sensor/camera.urdf.xacro (robot description, xacro)
@@ -33,4 +33,5 @@
             <xacro:box_inertia m="0.1" w="0.02" h="0.10" d="0.02" />
         </link>
+        <link name="camera_optical_link"></link>
         <joint name="camera_joint" type="fixed">
             <parent link="base_link"/>
@@ -38,4 +39,9 @@
             <origin xyz="${xyz}" rpy="0.0 0.0 0.0"/>
         </joint>
+        <joint name="camera_optical_joint" type="fixed">
+            <parent link="camera_link"/>
+            <child link="camera_optical_link"/>
+            <origin xyz="0 0 0" rpy="${-pi/2} 0.0 ${-pi/2}"/>
+        </joint>
     </xacro:macro>
 </robot>
